File: hw/sch_pcb/ISM02A.kicad_pcb (KiCad board)
At the start: 2 copper layers, 60.5 x 50.3 mm, 58 parts, among them J1 JUMP_3X2, J10 HEADER_2x01_PARALLEL, J11 HEADER_2x01_PARALLEL, J12 SMA, J13 U.FL, J14 SMA, J15 U.FL, J16 BMI-S-204-F, J2 SM07B-GHS-TB, J3 HEADER_2x01_PARALLEL, J4 HEADER_2x01_PARALLEL, J5 HEADER_2x01_PARALLEL, J6 HEADER_2x01_PARALLEL, J7 HEADER_2x01_PARALLEL, J8 HEADER_2x01_PARALLEL, J9 HEADER_2x01_PARALLEL, M1 HOLE, M2 HOLE, M3 HOLE, M4 HOLE, U1 SX1262, U2 MIC5504-3.3YM5, Y1 32MHz

Commit message: Documentation improvement.
Other:
- net class Default removed
- net class MLAB_power removed
