File: hw/sch_pcb/ISM02A.kicad_pcb (KiCad board)
At the start: 2 copper layers, 60.5 x 50.3 mm, 57 parts, among them J1 JUMP_3X2, J10 HEADER_2x01_PARALLEL, J11 HEADER_2x01_PARALLEL, J12 SMA, J13 HEADER_2x01_PARALLEL, J14 SMA, J15 HEADER_2x01_PARALLEL, J2 HEADER_2x01_PARALLEL, J3 HEADER_2x01_PARALLEL, J4 HEADER_2x01_PARALLEL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

Commit message: Revert "Edit"
This reverts commit 3bfea5ab87054fd9b05002ed626080fed2685c40.
Parts:
- added J16: BMI-S-204-F, MYLIB:BMI-S-204-F, B.Cu at (160.5, 111.3)
- J13, J15: value HEADER_2x01_PARALLEL -> U.FL; footprint Mlab_Pin_Headers:Straight_2x01 -> Connector_Coaxial:U.FL_Hirose_U.FL-R-SMT-1_Vertical
- J2: value HEADER_2x01_PARALLEL -> SM07B-GHS-TB; footprint Mlab_Pin_Headers:Straight_2x01 -> Connector_JST:JST_GH_SM07B-GHS-TB_1x07-1MP_P1.25mm_Horizontal
- moved J13 49.3 mm to (188.0, 118.0), turned to -90 degrees
- moved J15 33.1 mm to (188.0, 92.0), turned to 90 degrees
- moved J2 6.23 mm to (159.0, 82.3)
Connections:
- J13 pad 1: +3V3 -> Net-(C22-Pad2)
- J13 pad 2: +3V3 -> GND
- J15 pad 1: GND -> Net-(C23-Pad2)
- J2 pad 1: GND -> +5V
- J2 pad 2: GND -> /SCK
- U2 pad 4: (no net) -> Net-(U2-Pad4)
