File: hw/sch_pcb/ISM02B.kicad_sch (KiCad schematic)
At the start: 58 parts, among them J1 JUMP_3X2, J10 HEADER_2x01_PARALLEL, J11 HEADER_2x01_PARALLEL, J12 SMA, J13 U.FL, J14 SMA, J15 U.FL, J16 BMI-S-204-F, J2 SM07B-GHS-TB, J3 HEADER_2x01_PARALLEL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

Commit message: Edit
Parts:
- removed C18: 39pF, Capacitor_SMD:C_0603_1608Metric_Pad1.05x0.95mm_HandSolder, symbol ISM02A-rescue:C-Device-ISM02A-rescue
- removed C20, C23: 3p3, Capacitor_SMD:C_0603_1608Metric_Pad1.05x0.95mm_HandSolder, symbol ISM02A-rescue:C-Device-ISM02A-rescue
- removed J13, J15: U.FL, Connector_Coaxial:U.FL_Hirose_U.FL-R-SMT-1_Vertical, symbol ISM02A-rescue:SMA-MLAB_CONNECTORS
- removed J14: SMA, Mlab_CON:SMA6251A13G50, symbol ISM02A-rescue:SMA-MLAB_CONNECTORS
- removed J16: BMI-S-204-F, MYLIB:BMI-S-204-F, symbol ISM02A-rescue:RF_Shield_Two_Pieces-device
- removed J2: SM07B-GHS-TB, Connector_JST:JST_GH_SM07B-GHS-TB_1x07-1MP_P1.25mm_Horizontal, symbol ISM02A-rescue:SM07B-GHS-TB-MLAB_CONNECTORS_JST-ISM02A-rescue
- removed L8: 9n1, Inductor_SMD:L_0402_1005Metric, symbol ISM02A-rescue:L-Device-ISM02A-rescue
- added C?: 1nF, symbol Device:C
- added J13, J15, J2: HEADER_2x01_PARALLEL, Mlab_Pin_Headers:Straight_2x01, symbol ISM02A-rescue:HEADER_2x01_PARALLEL-MLAB_HEADER
- added R?: 100R, symbol Device:R
- added U?: PE4259, Package_TO_SOT_SMD:SOT-363_SC-70-6, symbol MLAB_IO:PE4259
Connections:
- net +3V3: now also J13.1, J13.2, U?.6 (#CTRL)
- net DIO2: now also R?.2
- net GND: now also C?.2, J15.1, J15.2, J2.1, J2.2, U?.2 (GND)
- net at C16.1, L6.2: now also U?.1 (RF1); no longer C17.2
- net at C10.1, C12.1: now also U?.3 (RF2)
- new net: C17.2, U?.5 (RFC)
- new net: C?.1, R?.1, U?.4 (CTRL)
Other:
- note removed: "SPI - Dronecode Autopilot Connector Standard"
- moved on the sheet: C1, C10, C11, C12, C13, C14, C15, C16, C17, C19, C21, C22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

Commit message: Edit
Parts:
- C18: renamed from C?; footprint (none) -> Capacitor_SMD:C_0603_1608Metric_Pad1.05x0.95mm_HandSolder; UST_ID (none) -> 5c70984812875079b91f8bec
- R1: footprint Mlab_R:SMD-0805 -> Mlab_R:SMD-0603; UST_ID 5c70984612875079b91f899f -> 5c70984512875079b91f8962
- R2: renamed from R?; footprint (none) -> Mlab_R:SMD-0603; UST_ID (none) -> 5c70984512875079b91f8956
- U3: renamed from U?; UST_ID (none) -> 5face19b12875025b3977e15
Changed lines of the file:
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@@
   (symbol (lib_id "power:+3.3V") (at 207.01 111.76 0) (unit 1)
     (in_bom yes) (on_board yes)
-    (property "Reference" "#PWR?" (id 0) (at 207.01 115.57 0)
+    (property "Reference" "#PWR04" (id 0) (at 207.01 115.57 0)
       (effects (font (size 1.27 1.27)) hide)
     )
@@
   (symbol (lib_id "power:GND") (at 193.04 138.43 0) (unit 1)
     (in_bom yes) (on_board yes)
-    (property "Reference" "#PWR?" (id 0) (at 193.04 144.78 0)
+    (property "Reference" "#PWR01" (id 0) (at 193.04 144.78 0)
       (effects (font (size 1.524 1.524)) hide)
     )
@@
   (symbol (lib_id "power:GND") (at 210.82 154.94 0) (unit 1)
     (in_bom yes) (on_board yes)
-    (property "Reference" "#PWR?" (id 0) (at 210.82 161.29 0)
+    (property "Reference" "#PWR05" (id 0) (at 210.82 161.29 0)
       (effects (font (size 1.524 1.524)) hide)
     )
@@
       (effects (font (size 1.27 1.27)) (justify left))
     )
-    (property "Footprint" "Mlab_R:SMD-0805" (id 2) (at 65.532 82.55 90)
+    (property "Footprint" "Mlab_R:SMD-0603" (id 2) (at 65.532 82.55 90)
       (effects (font (size 1.27 1.27)) hide)
     )
@@
       (effects (font (size 1.27 1.27)) hide)
     )
-    (property "UST_ID" "5c70984612875079b91f899f" (id 4) (at -24.13 166.37 0)
+    (property "UST_ID" "5c70984512875079b91f8962" (id 4) (at -24.13 166.37 0)
       (effects (font (size 1.27 1.27)) hide)
     )
@@
   (symbol (lib_id "Device:R") (at 220.98 144.78 90) (unit 1)
     (in_bom yes) (on_board yes)
-    (property "Reference" "R?" (id 0) (at 220.98 139.5538 90))
+    (property "Reference" "R2" (id 0) (at 220.98 139.5538 90))
     (property "Value" "100R" (id 1) (at 220.98 141.853 90))
-    (property "Footprint" "" (id 2) (at 220.98 146.558 90)
+    (property "Footprint" "Mlab_R:SMD-0603" (id 2) (at 220.98 146.558 90)
       (effects (font (size 1.27 1.27)) hide)
     )
@@
       (effects (font (size 1.27 1.27)) hide)
     )
+    (property "UST_ID" "5c70984512875079b91f8956" (id 4) (at 220.98 144.78 0)
+      (effects (font (size 1.27 1.27)) hide)
+    )
     (pin "1")
     (pin "2")
@@
       (effects (font (size 1.27 1.27)) hide)
     )
-    (property "Datasheet" "~" (id 3) (at 96.52 73.66 0)
+    (property "Datasheet" "" (id 3) (at 96.52 73.66 0)
       (effects (font (size 1.27 1.27)) hide)
     )
@@
   (symbol (lib_id "Device:C") (at 210.82 149.86 0) (unit 1)
     (in_bom yes) (on_board yes)
-    (property "Reference" "C?" (id 0) (at 213.7411 148.7106 0)
+    (property "Reference" "C18" (id 0) (at 213.7411 148.7106 0)
       (effects (font (size 1.27 1.27)) (justify left))
     )
@@
       (effects (font (size 1.27 1.27)) (justify left))
     )
-    (property "Footprint" "" (id 2) (at 211.7852 153.67 0)
+    (property "Footprint" "Capacitor_SMD:C_0603_1608Metric_Pad1.05x0.95mm_HandSolder" (id 2) (at 211.7852 153.67 0)
       (effects (font (size 1.27 1.27)) hide)
     )
     (property "Datasheet" "~" (id 3) (at 210.82 149.86 0)
+      (effects (font (size 1.27 1.27)) hide)
+    )
+    (property "UST_ID" "5c70984812875079b91f8bec" (id 4) (at 210.82 149.86 0)
       (effects (font (size 1.27 1.27)) hide)
     )
@@
   (symbol (lib_id "MLAB_IO:PE4259") (at 193.04 124.46 0) (mirror y) (unit 1)
     (in_bom yes) (on_board yes)
-    (property "Reference" "U?" (id 0) (at 193.04 110.0898 0))
+    (property "Reference" "U3" (id 0) (at 193.04 110.0898 0))
     (property "Value" "PE4259" (id 1) (at 193.04 112.3885 0))
     (property "Footprint" "Package_TO_SOT_SMD:SOT-363_SC-70-6" (id 2) (at 193.04 135.89 0)
@@
     )
     (property "Datasheet" "https://www.psemi.com/pdf/datasheets/pe4259ds.pdf" (id 3) (at 194.31 119.38 0)
+      (effects (font (size 1.27 1.27)) hide)
+    )
+    (property "UST_ID" "5face19b12875025b3977e15" (id 4) (at 193.04 124.46 0)
       (effects (font (size 1.27 1.27)) hide)
     )
@@
   )
   (symbol_instances
+    (path "/9eb5d852-8ece-4b0a-bdc4-48fcdb78ecfe"
+      (reference "#PWR01") (unit 1) (value "GND") (footprint "")
+    )
     (path "/00000000-0000-0000-0000-0000549d73b2"
       (reference "#PWR02") (unit 1) (value "GND") (footprint "")
@@
       (reference "#PWR03") (unit 1) (value "GND") (footprint "")
     )
+    (path "/f27cfdde-84b1-4904-bddc-8bf971fcd1ef"
+      (reference "#PWR04") (unit 1) (value "+3.3V") (footprint "")
+    )
+    (path "/af4624f3-4117-4d8a-94d5-cdea0d50f4be"
+      (reference "#PWR05") (unit 1) (value "GND") (footprint "")
+    )
     (path "/00000000-0000-0000-0000-00005da75df0"
       (reference "#PWR0101") (unit 1) (value "+5V") (footprint "")
@@
       (reference "#PWR0132") (unit 1) (value "GND") (footprint "")
     )
-    (path "/9eb5d852-8ece-4b0a-bdc4-48fcdb78ecfe"
-      (reference "#PWR?") (unit 1) (value "GND") (footprint "")
-    )
-    (path "/af4624f3-4117-4d8a-94d5-cdea0d50f4be"
-      (reference "#PWR?") (unit 1) (value "GND") (footprint "")
-    )
-    (path "/f27cfdde-84b1-4904-bddc-8bf971fcd1ef"
-      (reference "#PWR?") (unit 1) (value "+3.3V") (footprint "")
-    )
     (path "/00000000-0000-0000-0000-00005da84b07"
       (reference "C1") (unit 1) (value "-") (footprint "Capacitor_SMD:C_0603_1608Metric_Pad1.05x0.95mm_HandSolder")
@@
       (reference "C17") (unit 1) (value "39pF") (footprint "Capacitor_SMD:C_0603_1608Metric_Pad1.05x0.95mm_HandSolder")
     )
+    (path "/b327dba9-1654-4985-bb21-01143437b9a3"
+      (reference "C18") (unit 1) (value "1nF") (footprint "Capacitor_SMD:C_0603_1608Metric_Pad1.05x0.95mm_HandSolder")
+    )
     (path "/00000000-0000-0000-0000-00005dac3c31"
       (reference "C19") (unit 1) (value "3p3") (footprint "Capacitor_SMD:C_0603_1608Metric_Pad1.05x0.95mm_HandSolder")
@@
       (reference "C25") (unit 1) (value "10uF") (footprint "Mlab_R:SMD-0805")
     )
-    (path "/b327dba9-1654-4985-bb21-01143437b9a3"
-      (reference "C?") (unit 1) (value "1nF") (footprint "")
-    )
     (path "/00000000-0000-0000-0000-00005b4de0b5"
       (reference "D1") (unit 1) (value "BZV55C-5,6V") (footprint "Mlab_D:Diode-MiniMELF_Standard")
@@
     )
     (path "/00000000-0000-0000-0000-00005da81670"
-      (reference "R1") (unit 1) (value "10k") (footprint "Mlab_R:SMD-0805")
+      (reference "R1") (unit 1) (value "10k") (footprint "Mlab_R:SMD-0603")
     )
     (path "/fd608dde-7b8a-4217-a530-5ef4e2503818"
-      (reference "R?") (unit 1) (value "100R") (footprint "")
+      (reference "R2") (unit 1) (value "100R") (footprint "Mlab_R:SMD-0603")
     )
     (path "/00000000-0000-0000-0000-00005da52347"
@@
     )
     (path "/d5b16bba-6de8-45db-b493-dfea34cb144c"
-      (reference "U?") (unit 1) (value "PE4259") (footprint "Package_TO_SOT_SMD:SOT-363_SC-70-6")
+      (reference "U3") (unit 1) (value "PE4259") (footprint "Package_TO_SOT_SMD:SOT-363_SC-70-6")
     )
     (path "/00000000-0000-0000-0000-00005db3724c"

Commit message: Edit
Parts:
- J12: value SMA -> MCX; footprint Mlab_CON:SMA6251A13G50 -> Mlab_CON:MCX; UST_ID 5c70984412875079b91f87ac -> (none)
Changed lines of the file:
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@@
       (effects (font (size 1.524 1.524)) (justify left))
     )
-    (property "Value" "SMA" (id 1) (at 259.7912 124.0536 0)
+    (property "Value" "MCX" (id 1) (at 259.7912 124.0536 0)
       (effects (font (size 1.524 1.524)) (justify left))
     )
-    (property "Footprint" "Mlab_CON:SMA6251A13G50" (id 2) (at 255.27 121.92 0)
+    (property "Footprint" "Mlab_CON:MCX" (id 2) (at 255.27 121.92 0)
       (effects (font (size 1.524 1.524)) hide)
     )
@@
       (effects (font (size 1.524 1.524)))
     )
-    (property "UST_ID" "5c70984412875079b91f87ac" (id 4) (at 6.35 208.28 0)
+    (property "UST_ID" "" (id 4) (at 6.35 208.28 0)
       (effects (font (size 1.27 1.27)) hide)
     )
@@
     )
     (path "/00000000-0000-0000-0000-00005da75a91"
-      (reference "J12") (unit 1) (value "SMA") (footprint "Mlab_CON:SMA6251A13G50")
+      (reference "J12") (unit 1) (value "MCX") (footprint "Mlab_CON:MCX")
     )
     (path "/5f0a40cb-3afe-432c-bba8-05e0afefaf7c"
