File: hw/sch_pcb/ISM02B.kicad_pcb (KiCad board)
At the start: 2 copper layers, 60.5 x 50.3 mm, 58 parts, among them J1 JUMP_3X2, J10 HEADER_2x01_PARALLEL, J11 HEADER_2x01_PARALLEL, J12 SMA, J13 U.FL, J14 SMA, J15 U.FL, J16 BMI-S-204-F, J2 SM07B-GHS-TB, J3 HEADER_2x01_PARALLEL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

Commit message: Edit
Parts:
- removed J16: BMI-S-204-F, MYLIB:BMI-S-204-F
- J13, J15: value U.FL -> HEADER_2x01_PARALLEL; footprint Connector_Coaxial:U.FL_Hirose_U.FL-R-SMT-1_Vertical -> Mlab_Pin_Headers:Straight_2x01
- J2: value SM07B-GHS-TB -> HEADER_2x01_PARALLEL; footprint Connector_JST:JST_GH_SM07B-GHS-TB_1x07-1MP_P1.25mm_Horizontal -> Mlab_Pin_Headers:Straight_2x01
- moved J13 49.3 mm to (166.9, 73.4), turned to 0 degrees
- moved J15 33.1 mm to (160.6, 73.4), turned to 0 degrees
- moved J2 6.23 mm to (160.3, 76.2)
Connections:
- J13 pad 1: Net-(C22-Pad2) -> +3V3
- J13 pad 2: GND -> +3V3
- J15 pad 1: Net-(C23-Pad2) -> GND
- J2 pad 1: +5V -> GND
- J2 pad 2: /SCK -> GND
- U2 pad 4: Net-(U2-Pad4) -> (no net)

Commit message: Edit
Parts:
- removed C20, C23: 3p3, Capacitor_SMD:C_0603_1608Metric_Pad1.05x0.95mm_HandSolder
- removed J14: SMA, Mlab_CON:SMA6251A13G50
- removed L8: 9n1, Inductor_SMD:L_0402_1005Metric
- added R2: 100R, Mlab_R:SMD-0603, B.Cu at (167.7, 116.0)
- added U3: PE4259, Package_TO_SOT_SMD:SOT-363_SC-70-6, B.Cu at (165.1, 115.9)
- C18: value 39pF -> 1nF
- R1: footprint Mlab_R:SMD-0805 -> Mlab_R:SMD-0603
- moved J13 50.7 mm to (139.2, 115.8)
- moved J2 47.1 mm to (139.2, 118.4)
- moved J15 45.3 mm to (139.2, 113.3)
- moved J1 29.0 mm to (126.7, 118.4)
- moved M1 22.7 mm to (180.3, 104.1)
- moved M2 20.3 mm to (139.7, 104.1)
- moved J11 16.0 mm to (160.0, 104.1)
- moved R1 16.0 mm to (161.8, 113.4)
- moved J10 16.0 mm to (152.4, 104.1)
- moved J3 16.0 mm to (162.6, 104.1)
- moved J4 16.0 mm to (171.7, 104.1)
- moved J5 16.0 mm to (166.6, 104.1)
- moved J6 16.0 mm to (169.1, 104.1)
- moved J7 16.0 mm to (174.2, 104.1)
- moved J8 16.0 mm to (157.5, 104.1)
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Connections:
- C17 pad 2: Net-(C16-Pad1) -> Net-(U3-Pad5)
- C18 pad 2: Net-(C10-Pad1) -> GND
Routing:
- net GND: track 685.2 -> 44.9 mm, vias 309 -> 27
- net +5V: track 53.7 -> 9.59 mm, vias 1 -> 0
- net Net-(C23-Pad2): track 28.7 -> 0.00 mm
- net /#CS: track 37.3 -> 24.1 mm, vias 1 -> 0
- net /BUSY: track 22.8 -> 11.2 mm
- net Net-(C22-Pad2): track 12.6 -> 1.53 mm
- net +3V3: track 37.7 -> 28.1 mm
- net Net-(C8-Pad1): track 5.31 -> 13.1 mm, vias 0 -> 1
- net /MOSI: track 28.7 -> 21.4 mm, vias 1 -> 0
- net /SCK: track 29.6 -> 23.6 mm
- net /MISO: track 25.0 -> 21.1 mm
- net Net-(C17-Pad1): track 5.19 -> 1.56 mm
- net Net-(C13-Pad1): track 5.40 -> 1.86 mm
- net Net-(C18-Pad1): track 3.26 -> 0.00 mm
- net Net-(C16-Pad1): track 3.06 -> 0.00 mm
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Other:
- board text removed: "RF IN"

Commit message: Edit
Other:
- board size 60.5 x 50.3 mm -> 50.3 x 30 mm
Changed lines of the file:
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@@
     )
   )
-  (gr_line (start 134.874 129.286) (end 134.874 78.994) (layer "Edge.Cuts") (width 0.15))
-  (gr_line (start 134.874 78.994) (end 195.326 78.994) (layer "Edge.Cuts") (width 0.15))
-  (gr_line (start 195.326 129.286) (end 134.874 129.286) (layer "Edge.Cuts") (width 0.15))
-  (gr_line (start 195.326 78.994) (end 195.326 129.286) (layer "Edge.Cuts") (width 0.15))
+  (gr_line (start 134.874 99.314) (end 134.874 129.286) (layer "Edge.Cuts") (width 0.15))
+  (gr_line (start 134.874 99.314) (end 185.166 99.314) (layer "Edge.Cuts") (width 0.15))
+  (gr_line (start 185.166 129.286) (end 134.874 129.286) (layer "Edge.Cuts") (width 0.15))
+  (gr_line (start 185.166 129.286) (end 185.166 99.314) (layer "Edge.Cuts") (width 0.15))
   (gr_text "MISO\nMOSI\nSCK\nCS" (at 170.524 106.68 90) (layer "F.SilkS")
     (effects (font (size 1.5 1.5) (thickness 0.3)) (justify right))
@@
   (zone (net 2) (net_name "GND") (layer "B.Cu") (hatch edge 0.508)
     (connect_pads (clearance 0.265))
-    (min_thickness 0.254)
+    (min_thickness 0.254) (filled_areas_thickness no)
     (fill yes (thermal_gap 0.508) (thermal_bridge_width 0.508))
     (polygon
       (pts
-        (xy 134.874 78.994)
+        (xy 134.366 78.994)
         (xy 195.326 78.994)
         (xy 195.326 129.286)
-        (xy 134.874 129.286)
-      )
-    )
+        (xy 134.366 129.286)
+      )
+    )

Commit message: Edit
Parts:
- J12: value SMA -> MCX; footprint Mlab_CON:SMA6251A13G50 -> Mlab_CON:MCX
- moved C2 26.4 mm to (146.1, 111.3), turned to 0 degrees
- moved C25 26.3 mm to (145.3, 108.6)
- moved J1 25.4 mm to (147.8, 104.1), turned to 90 degrees
- moved C21 22.6 mm to (143.0, 110.1), turned to -90 degrees
- moved U2 18.5 mm to (139.9, 110.1), turned to 180 degrees
- moved C24 14.2 mm to (136.7, 109.8), turned to 90 degrees
- moved C18 10.5 mm to (160.8, 112.1), turned to 180 degrees
- moved R2 7.33 mm to (163.2, 110.2), turned to 180 degrees
- moved R1 6.27 mm to (167.2, 110.2)
- moved D1 4.85 mm to (149.6, 108.7), turned to 0 degrees
- moved C12 1.80 mm to (161.6, 116.1)
- moved C1 1.39 mm to (152.5, 124.5)
- moved C3 1.39 mm to (147.3, 124.5)
- moved Y1 1.39 mm to (149.9, 126.1)
- moved C8 1.35 mm to (158.5, 115.3)
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Routing:
- net +3V3: track 28.1 -> 65.0 mm, vias 4 -> 5
- net GND: track 44.9 -> 58.8 mm, vias 27 -> 183
- net /#RESET: track 17.8 -> 30.8 mm, vias 0 -> 1
- net /DIO2: track 17.5 -> 27.0 mm, vias 0 -> 1
- net +5V: track 9.59 -> 18.8 mm
- net /BUSY: track 11.2 -> 19.6 mm
- net Net-(C18-Pad1): track 0.00 -> 7.64 mm, vias 0 -> 2
- net Net-(C22-Pad2): track 1.53 -> 8.56 mm
- net /#CS: track 24.1 -> 30.8 mm
- net Net-(C8-Pad1): track 13.1 -> 6.65 mm, vias 1 -> 0
- net /DIO3: track 23.1 -> 29.1 mm
- net /MOSI: track 21.4 -> 26.6 mm
- net /SCK: track 23.6 -> 28.3 mm
- net /MISO: track 21.1 -> 25.5 mm
- net Net-(C16-Pad1): track 0.00 -> 4.18 mm
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- removed copper zone on B.Cu, net Net-(C4-Pad1)
Other:
- board text added: "#CS"
- board text added: "#RESET"
- board text added: "2021"
- board text added: "3V3"
- board text added: "BUSY"
- board text added: "DIO1"
- board text added: "DIO2"
- board text added: "DIO3"
- board text added: "IN 5V"
- board text added: "MISO"
- board text added: "MLAB.CZ ISM02B"
- board text added: "MOSI"
- board text added: "SCK"
- board text removed: "2019"
- board text removed: "5V"
- board text removed: "DIO3 DIO2 DIO1 BUSY RESET"
- board text removed: "MISO MOSI SCK CS"
- board text removed: "MLAB.CZ - ISM02A"

Commit message: Edit
Other:
- board text added: "IN/OUT"
- board text added: "RF"
- board text removed: "RF OUT"
Changed lines of the file:
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@@
     (property "UST_ID" "")
     (attr through_hole)
-    (fp_text reference "J12" (at 0 -5.1 90) (layer "F.SilkS")
+    (fp_text reference "J12" (at 0 -5.1 90) (layer "F.SilkS") hide
       (effects (font (size 1.5 1.5) (thickness 0.15)))
     )
@@
     (effects (font (size 1.5 1.5) (thickness 0.3)))
   )
-  (gr_text " RF OUT" (at 170.18 88.9) (layer "F.SilkS")
-    (effects (font (size 1.5 1.5) (thickness 0.3)) (justify left))
+  (gr_text "IN/OUT" (at 179.3748 120.015) (layer "F.SilkS")
+    (effects (font (size 1.5 1.5) (thickness 0.3)))
   )
   (gr_text "2021" (at 155.448 125.984) (layer "F.SilkS")
@@
   (gr_text "#RESET" (at 163.556 106.68 90) (layer "F.SilkS")
     (effects (font (size 1.5 1.5) (thickness 0.3)) (justify right))
+  )
+  (gr_text "RF" (at 179.3748 109.22) (layer "F.SilkS")
+    (effects (font (size 1.5 1.5) (thickness 0.3)))
   )
   (gr_text "MOSI" (at 169.642 106.68 90) (layer "F.SilkS")
@@
   (via (at 153.67 100.33) (size 0.6) (drill 0.3) (layers "F.Cu" "B.Cu") (free) (net 2))
   (via (at 169.164 116.967) (size 0.6) (drill 0.3) (layers "F.Cu" "B.Cu") (free) (net 2))
-  (via (at 178.435 108.585) (size 0.6) (drill 0.3) (layers "F.Cu" "B.Cu") (free) (net 2))
+  (via (at 177.8 108.585) (size 0.6) (drill 0.3) (layers "F.Cu" "B.Cu") (free) (net 2))
   (via (at 170.053 111.633) (size 0.6) (drill 0.3) (layers "F.Cu" "B.Cu") (free) (net 2))
   (via (at 172.085 128.27) (size 0.6) (drill 0.3) (layers "F.Cu" "B.Cu") (free) (net 2))
@@
   (via (at 160.655 113.919) (size 0.6) (drill 0.3) (layers "F.Cu" "B.Cu") (free) (net 2))
   (via (at 150.876 122.301) (size 0.6) (drill 0.3) (layers "F.Cu" "B.Cu") (net 2))
-  (via (at 180.975 120.015) (size 0.6) (drill 0.3) (layers "F.Cu" "B.Cu") (free) (net 2))
+  (via (at 181.61 120.015) (size 0.6) (drill 0.3) (layers "F.Cu" "B.Cu") (free) (net 2))
   (via (at 159.766 122.809) (size 0.6) (drill 0.3) (layers "F.Cu" "B.Cu") (free) (net 2))
   (via (at 149.858 123.86) (size 0.6) (drill 0.3) (layers "F.Cu" "B.Cu") (net 2))
@@
   (via (at 177.8 100.33) (size 0.6) (drill 0.3) (layers "F.Cu" "B.Cu") (free) (net 2))
   (via (at 175.26 100.33) (size 0.6) (drill 0.3) (layers "F.Cu" "B.Cu") (free) (net 2))
-  (via (at 177.165 108.585) (size 0.6) (drill 0.3) (layers "F.Cu" "B.Cu") (free) (net 2))
+  (via (at 176.53 108.585) (size 0.6) (drill 0.3) (layers "F.Cu" "B.Cu") (free) (net 2))
   (via (at 146.939 112.649) (size 0.6) (drill 0.3) (layers "F.Cu" "B.Cu") (free) (net 2))
   (via (at 158.115 128.27) (size 0.6) (drill 0.3) (layers "F.Cu" "B.Cu") (free) (net 2))
@@
   (via (at 167.64 100.33) (size 0.6) (drill 0.3) (layers "F.Cu" "B.Cu") (free) (net 2))
   (via (at 173.99 100.33) (size 0.6) (drill 0.3) (layers "F.Cu" "B.Cu") (free) (net 2))
-  (via (at 182.245 120.015) (size 0.6) (drill 0.3) (layers "F.Cu" "B.Cu") (free) (net 2))
+  (via (at 183.515 120.015) (size 0.6) (drill 0.3) (layers "F.Cu" "B.Cu") (free) (net 2))
   (via (at 148.908011 121.145981) (size 0.6) (drill 0.3) (layers "F.Cu" "B.Cu") (net 2))
   (via (at 148.59 100.33) (size 0.6) (drill 0.3) (layers "F.Cu" "B.Cu") (free) (net 2))
@@
   (via (at 184.15 107.95) (size 0.6) (drill 0.3) (layers "F.Cu" "B.Cu") (free) (net 2))
   (via (at 171.704 116.967) (size 0.6) (drill 0.3) (layers "F.Cu" "B.Cu") (free) (net 2))
-  (via (at 179.705 120.015) (size 0.6) (drill 0.3) (layers "F.Cu" "B.Cu") (free) (net 2))
-  (via (at 178.435 120.015) (size 0.6) (drill 0.3) (layers "F.Cu" "B.Cu") (free) (net 2))
+  (via (at 179.705 118.745) (size 0.6) (drill 0.3) (layers "F.Cu" "B.Cu") (free) (net 2))
+  (via (at 179.07 120.015) (size 0.6) (drill 0.3) (layers "F.Cu" "B.Cu") (free) (net 2))
   (via (at 166.497 121.158) (size 0.6) (drill 0.3) (layers "F.Cu" "B.Cu") (free) (net 2))
   (via (at 160.02 100.33) (size 0.6) (drill 0.3) (layers "F.Cu" "B.Cu") (free) (net 2))
@@
   (via (at 175.006 115.062) (size 0.6) (drill 0.3) (layers "F.Cu" "B.Cu") (free) (net 2))
   (via (at 135.89 118.11) (size 0.6) (drill 0.3) (layers "F.Cu" "B.Cu") (free) (net 2))
-  (via (at 177.165 120.015) (size 0.6) (drill 0.3) (layers "F.Cu" "B.Cu") (free) (net 2))
+  (via (at 177.8 120.015) (size 0.6) (drill 0.3) (layers "F.Cu" "B.Cu") (free) (net 2))
   (via (at 141.859 107.569) (size 0.6) (drill 0.3) (layers "F.Cu" "B.Cu") (net 2))
   (via (at 163.83 111.633) (size 0.6) (drill 0.3) (layers "F.Cu" "B.Cu") (free) (net 2))
@@
   (via (at 156.845 128.27) (size 0.6) (drill 0.3) (layers "F.Cu" "B.Cu") (free) (net 2))
   (via (at 167.132 122.428) (size 0.6) (drill 0.3) (layers "F.Cu" "B.Cu") (free) (net 2))
-  (via (at 179.705 108.585) (size 0.6) (drill 0.3) (layers "F.Cu" "B.Cu") (free) (net 2))
+  (via (at 179.07 110.49) (size 0.6) (drill 0.3) (layers "F.Cu" "B.Cu") (free) (net 2))
   (via (at 150.876 128.27) (size 0.6) (drill 0.3) (layers "F.Cu" "B.Cu") (net 2))
   (via (at 146.05 121.92) (size 0.6) (drill 0.3) (layers "F.Cu" "B.Cu") (free) (net 2))
