File: hw/sch_pcb/ISM02B.kicad_pcb (KiCad board)
At the start: 2 copper layers, 50.3 x 30 mm, 55 parts, among them J1 JUMP_3X2, J10 HEADER_2x01_PARALLEL, J11 HEADER_2x01_PARALLEL, J12 MCX, J13 HEADER_2x01_PARALLEL, J15 HEADER_2x01_PARALLEL, J2 HEADER_2x01_PARALLEL, J3 HEADER_2x01_PARALLEL, J4 HEADER_2x01_PARALLEL, J5 HEADER_2x01_PARALLEL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

Commit message: kicad 7
Routing:
- net GND: track 58.8 -> 55.2 mm
- net Net-(C10-Pad1): track 5.15 -> 4.61 mm
